Commit message: adding new script configurations for face recognition and gripper deployment to catch object step by step and start exploring contact plugin for gripper

File: robot-face-recognition-project/the_robot_description/urdf/modelNOUV.xacro (robot description, xacro)
@@ -380,5 +380,5 @@
           </contact>
         </surface>
-    <collision name="the_robot__collision">
+    <collision name="left_finger__collision">
       <!--<origin rpy="0 0 0" xyz="0.5 -0.8 0.05"/>-->
       <geometry>
@@ -393,4 +393,10 @@
       </geometry>
     </visual>
+    <!--<sensor name='my_contact_the_robot__left_finger' type='contact'>
+      <contact>
+        <collision>the_robot__left_finger_collision</collision>
+      </contact>
+      <update_rate> 5 </update_rate>
+    </sensor>-->
   </link>
   <link name="the_robot__left_finger_tip">
