Commit message: adding new urdf configurations

File: robot-face-recognition-project/the_robot_description/urdf/model.xacro (robot description, xacro)
@@ -393,10 +393,10 @@
       </geometry>
     </visual>
-    <sensor name='my_contact_the_robot__left_finger' type='contact'>
+    <!--<sensor name='my_contact_the_robot__left_finger' type='contact'>
       <contact>
         <collision>the_robot__left_finger_collision</collision>
       </contact>
       <update_rate> 5 </update_rate>
-    </sensor>
+    </sensor>-->
   </link>
   <link name="the_robot__left_finger_tip">

File: robot-face-recognition-project/the_robot_description/urdf/test_collision/modelNOUV.xacro (robot description, xacro)
@@ -161,5 +161,5 @@
     <parent link="the_robot__riser"/>
     <child link="the_robot__palm"/>
-    <origin rpy="0 0 0" xyz="0  0   -0.1"/>
+    <origin rpy="0 0 0" xyz="0  0   -0.4"/>
     <axis xyz="0 0 1"/>
     <limit effort="1000.0" lower="0.0" upper="0.9" velocity="1000.0"/>
@@ -205,5 +205,5 @@
     <parent link="the_robot__palm"/>
     <child link="the_robot__hokuyo_link"/>
-    <origin rpy="0 0 0" xyz="0  0    -0.2"/>
+    <origin rpy="0 0 0" xyz="0  0    0.2"/>
     <axis xyz="0 0 0"/>
     <limit effort="0" lower="0" upper="0" velocity="0"/>
@@ -393,11 +393,24 @@
       </geometry>
     </visual>
-    <sensor name='my_contact_the_robot__left_finger' type='contact'>
+    <!--<sensor name='my_contact_the_robot__left_finger' type='contact'>
       <contact>
         <collision>the_robot__left_finger_collision</collision>
       </contact>
       <update_rate> 5 </update_rate>
-    </sensor>
-  </link>
+    </sensor>-->
+  </link>
+ <gazebo reference="the_robot__left_finger">
+    <sensor name='my_contact_the_robot__left_finger' type='contact'>
+      <plugin name="my_plugin" filename="libcontact.so"/>
+        <always_on>true</always_on>
+        <contact>
+          <collision>the_robot__left_finger_fixed_joint_lump__left_finger__collision_collision</collision>
+          <!--<collision>__default__</collision>-->
+          <!--<collision>the_robot__left_finger_fixed_joint_lump__left_finger__collision_collision</collision>-->
+          <topic>__default_topic__</topic>
+        </contact>
+        <update_rate> 5 </update_rate>
+     </sensor>
+  </gazebo>
   <link name="the_robot__left_finger_tip">
     <inertial>

File: robot-face-recognition-project/the_robot_description/urdf/test_collision/robot.urdf (robot description, URDF)
Before this commit: robot the_robot, 13 links, 12 joints
Joints:
- joint the_robot__hokuyo_joint: origin xyz=0  0    -0.2 rpy=0 0 0 -> xyz=0  0    0.2 rpy=0 0 0
- joint the_robot__palm_riser: origin xyz=0  0   -0.1 rpy=0 0 0 -> xyz=0  0   -0.4 rpy=0 0 0
